File: Claw10 PCB.kicad_pcb (KiCad board)
At the start: 2 copper layers, 24 parts, among them SW1 SW_Push, U1 ATmega32U4-AU, Y1 16MHz

Commit message: 4/3/20
Parts:
- C1, C2, C3, C4, C5, C6, C7, D1, D2, D3, D4, F1, MX1, MX2, MX3, MX4, R1, R2, R3, R4, SW1, U1, USB1, Y1: moved to B.Cu
- moved C1 122.7 mm to (43.4, 54.0), turned to 90 degrees
- moved R2 114.3 mm to (47.5, 32.7), turned to 90 degrees
- moved USB1 109.0 mm to (46.8, 19.5), turned to 270 degrees
- moved C5 106.6 mm to (37.0, 42.8)
- moved C6 102.5 mm to (43.4, 47.4), turned to 270 degrees
- moved R1 100.4 mm to (45.5, 32.6), turned to 90 degrees
- moved F1 99.7 mm to (43.3, 32.8), turned to 90 degrees
- moved C2 98.7 mm to (63.1, 31.5), turned to 270 degrees
- moved C7 96.8 mm to (53.6, 63.8)
- moved C3 96.2 mm to (52.6, 31.4), turned to 270 degrees
- moved C4 93.7 mm to (61.8, 63.8), turned to 180 degrees
- moved Y1 88.4 mm to (58.0, 31.5), turned to 180 degrees
- moved R3 82.2 mm to (66.8, 62.9)
- moved U1 80.7 mm to (59.3, 51.8)
- moved SW1 73.2 mm to (70.2, 33.7), turned to 90 degrees
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Routing:
- net ROW1: track 0.00 -> 67.1 mm
- net ROW0: track 0.00 -> 59.5 mm
- net COL0: track 0.00 -> 38.6 mm
- net COL1: track 0.00 -> 19.1 mm
- net Net-(D2-Pad2): track 0.00 -> 13.9 mm
- net Net-(D1-Pad2): track 0.00 -> 13.9 mm
- net Net-(D4-Pad2): track 0.00 -> 12.1 mm
- net Net-(D3-Pad2): track 0.00 -> 12.1 mm
Other:
- net class Default: trace_width 0.25 -> 0.254
- net class power added: clearance 0.2, trace_width 0.381, via_dia 0.8, via_drill 0.4

Commit message: 4/3/20 v2
Parts:
- moved R4 13.9 mm to (66.3, 54.7), turned to 90 degrees
- moved C5 7.78 mm to (44.6, 41.5), turned to 180 degrees
- moved SW1 7.00 mm to (69.1, 40.6)
- moved U1 5.45 mm to (56.8, 47.0)
- moved C1 2.46 mm to (43.6, 51.6)
- moved C6 0.98 mm to (43.6, 46.4)
- turned C4 to 90 degrees
- turned C7 to 90 degrees
- turned R3 to 90 degrees
Routing:
- net GND: track 0.49 -> 144.6 mm, vias 0 -> 5
- net Net-(R3-Pad2): track 0.00 -> 83.9 mm, vias 0 -> 4
- net +5V: track 0.36 -> 83.4 mm
- net Net-(R1-Pad1): track 0.00 -> 31.1 mm
- net Net-(C3-Pad1): track 0.00 -> 25.9 mm, vias 0 -> 2
- net COL1: track 19.1 -> 44.6 mm, vias 0 -> 2
- net Net-(R2-Pad1): track 0.00 -> 18.5 mm, vias 0 -> 2
- net ROW1: track 67.1 -> 84.5 mm
- net ROW0: track 59.5 -> 74.5 mm, vias 0 -> 2
- net Net-(C2-Pad2): track 0.00 -> 14.0 mm
- net COL0: track 38.6 -> 48.3 mm
- net VCC: track 0.00 -> 8.67 mm
- net D+: track 0.00 -> 8.03 mm
- net Net-(C6-Pad1): track 0.14 -> 8.14 mm
- net D-: track 0.00 -> 7.93 mm
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
Commit message: 4/3/20 v3
Routing:
- added copper zone on B.Cu, net GND
Other:
- board outline added: 73.7 x 50.8 mm
- board text added: "First ClawBoard Evah!"
